File: fx-WahWahWah.kicad_sch (KiCad schematic)
At the start: 40 parts, among them J1 Conn_01x10, Q1 2N5088, Q2 2N5089, SW1 ON-ON

Commit message: Fix DNP issues.
Parts:
- C21, C23, C24, C25, R21, R22, R23, R24, R25, R26, R27, R28, R29, R30: now not fitted
Changed lines of the file:
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@@
 		(on_board yes)
 		(in_pos_files yes)
-		(dnp no)
+		(dnp yes)
 		(property "Reference" "R25"
 			(at 109.474 114.3 90)
@@
 		(on_board yes)
 		(in_pos_files yes)
-		(dnp no)
+		(dnp yes)
 		(property "Reference" "R28"
 			(at 135.89 37.084 90)
@@
 		(on_board yes)
 		(in_pos_files yes)
-		(dnp no)
+		(dnp yes)
 		(property "Reference" "R26"
 			(at 118.11 84.074 90)
@@
 		(on_board yes)
 		(in_pos_files yes)
-		(dnp no)
+		(dnp yes)
 		(property "Reference" "R22"
 			(at 110.744 60.96 90)
@@
 		(on_board yes)
 		(in_pos_files yes)
-		(dnp no)
+		(dnp yes)
 		(property "Reference" "C25"
 			(at 147.066 54.61 90)
@@
 		(on_board yes)
 		(in_pos_files yes)
-		(dnp no)
+		(dnp yes)
 		(property "Reference" "C23"
 			(at 72.39 69.596 90)
@@
 		(on_board yes)
 		(in_pos_files yes)
-		(dnp no)
+		(dnp yes)
 		(property "Reference" "R29"
 			(at 48.514 97.79 90)
@@
 		(on_board yes)
 		(in_pos_files yes)
-		(dnp no)
+		(dnp yes)
 		(property "Reference" "C24"
 			(at 134.62 69.596 90)
@@
 		(on_board yes)
 		(in_pos_files yes)
-		(dnp no)
+		(dnp yes)
 		(property "Reference" "R23"
 			(at 82.042 67.564 90)
@@
 		(on_board yes)
 		(in_pos_files yes)
-		(dnp no)
+		(dnp yes)
 		(property "Reference" "C21"
 			(at 74.93 40.386 90)
@@
 		(on_board yes)
 		(in_pos_files yes)
-		(dnp no)
+		(dnp yes)
 		(property "Reference" "R30"
 			(at 166.624 36.83 90)
@@
 			(at 168.91 36.83 0)
 			(hide yes)
-			(show_name no)
+			(show_name yes)
 			(do_not_autoplace no)
 			(effects
@@
 		(on_board yes)
 		(in_pos_files yes)
-		(dnp no)
+		(dnp yes)
 		(property "Reference" "R27"
 			(at 96.774 38.1 90)
@@
 		(on_board yes)
 		(in_pos_files yes)
-		(dnp no)
+		(dnp yes)
 		(property "Reference" "R24"
 			(at 99.06 84.074 90)
@@
 		(on_board yes)
 		(in_pos_files yes)
-		(dnp no)
+		(dnp yes)
 		(property "Reference" "R21"
 			(at 64.77 42.164 90)

Commit message: Some final silk cleanups
Parts:
- C26: footprint Capacitor_THT:C_Rect_L7.2mm_W5.5mm_P5.00mm_FKS2_FKP2_MKS2_MKP2 -> Capacitor_THT:C_Rect_L7.2mm_W4.5mm_P5.00mm_FKS2_FKP2_MKS2_MKP2
Changed lines of the file:
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@@
 			)
 		)
-		(property "Footprint" "Capacitor_THT:C_Rect_L7.2mm_W5.5mm_P5.00mm_FKS2_FKP2_MKS2_MKP2"
+		(property "Footprint" "Capacitor_THT:C_Rect_L7.2mm_W4.5mm_P5.00mm_FKS2_FKP2_MKS2_MKP2"
 			(at 69.85 114.3 0)
 			(hide yes)

Commit message: fx-WahWahWah v0.3 fab outputs (g3)
Parts:
- removed J1: Conn_01x10, Connector_PinHeader_2.54mm:PinHeader_1x10_P2.54mm_Vertical, symbol Connector_Generic:Conn_01x10
- added J10, J11, J2, J3, J4, J5, J6, J7, J8, J9: Conn_01x01_Pin, TestPoint:Vector T46-5-9M, symbol Connector:Conn_01x01_Pin
Connections:
- net +9V: now also J8.1 (Pin_1)
- net BATT_NEG: now also J6.1 (Pin_1), J7.1 (Pin_1)
- net GND: now also J10.1 (Pin_1), J11.1 (Pin_1), J9.1 (Pin_1)
- net IN_JACK_TIP: now also J3.1 (Pin_1), J4.1 (Pin_1)
- net POT_LUG_2: now also J2.1 (Pin_1)
- net POT_LUG_3: now also J5.1 (Pin_1)
